Commit message: Rename URDF to so101_sroi.urdf and update camera link name
- Renamed so101_new_gripper_test.urdf to so101_sroi.urdf
- Updated robot name to so101_sroi
- Changed camera_mount_link to camera_link
- Changed camera_mount_joint to camera_joint
- Updated visualize_all.py to use new URDF path

Co-Authored-By: Claude Opus 4.6 <noreply@anthropic.com>

File: Simulation/SO101/so101_sroi.urdf (robot description, URDF)
Before this commit: robot so101_new_gripper_test, 7 links, 6 joints
Links:
- removed link camera_mount_link
- added link camera_link, mass 1e-9
Joints:
- removed joint camera_mount_joint
- added joint camera_joint: type fixed, parent gripper_link, child camera_link, origin xyz=0.046 0 -0.043 rpy=0 1.5708 0
