Commit message: Update mesh file paths in so101_sroi.urdf to relative references

File: Simulation/SO101/so101_sroi.urdf (robot description, URDF)
Before this commit: robot so101_sroi, 7 links, 6 joints
Links:
- link base_link: geometry collision mesh filename=assets/base_motor_holder_so101_v1.stl; collision mesh filename=assets/base_so101_v2.stl
- link gripper_link: geometry collision mesh filename=assets/Gripper_SROI.stl; visual mesh filename=assets/Gripper_SROI.stl
- link lower_arm_link: geometry collision mesh filename=assets/motor_holder_so101_wrist_v1.stl; collision mesh filename=assets/sts3215_03a_v1.stl
- link shoulder_link: geometry collision mesh filename=assets/motor_holder_so101_base_v1.stl; collision mesh filename=assets/rotation_pitch_so101_v1.stl
- link upper_arm_link: geometry collision mesh filename=assets/sts3215_03a_v1.stl; collision mesh filename=assets/upper_arm_so101_v1.stl
- link wrist_link: geometry collision mesh filename=assets/sts3215_03a_no_horn_v1.stl; collision mesh filename=assets/wrist_roll_pitch_so101_v2.stl

Commit message: Add gripper frame and moving jaw links with associated joints in so101_sroi.urdf

File: Simulation/SO101/so101_sroi.urdf (robot description, URDF)
Before this commit: robot so101_sroi, 7 links, 6 joints
Links:
- added link gripper_frame_link, mass 1e-9
- added link moving_jaw_so101_v1_link, mass 0.012; collision mesh filename=assets/moving_jaw_so101_v1.stl; visual mesh filename=assets/moving_jaw_so101_v1.stl
Joints:
- added joint gripper: type revolute, parent gripper_link, child moving_jaw_so101_v1_link, origin xyz=0.0202 0.0188 -0.0234 rpy=1.5708 -5.24284e-08 -1.41553e-15, axis 0 0 1, limit lower=-0.174533 upper=1.74533 effort=10 velocity=10
- added joint gripper_frame_joint: type fixed, parent gripper_link, child gripper_frame_link, origin xyz=-0.0079 -0.000218121 -0.0981274 rpy=0 3.14159 0, axis 0 0 0

Commit message: Remove visual and collision elements for moving jaw link and adjust camera joint orientation

File: Simulation/SO101/so101_sroi.urdf (robot description, URDF)
Before this commit: robot so101_sroi, 9 links, 8 joints
Links:
- link moving_jaw_so101_v1_link: geometry 
Joints:
- joint camera_joint: origin xyz=0.046 0 -0.043 rpy=0 1.5708 0 -> xyz=0.046 0 -0.043 rpy=0 1.8008 0

Commit message: Add OpenCV camera optical frame and adjust joint parameters for camera integration

File: Simulation/SO101/so101_sroi.urdf (robot description, URDF)
Before this commit: robot so101_sroi, 9 links, 8 joints
Links:
- added link camera_optical_link, mass 1e-9
Joints:
- added joint camera_optical_joint: type fixed, parent camera_link, child camera_optical_link, origin xyz=0 0 0 rpy=-1.57079632679 0 -1.57079632679
- joint camera_joint: origin xyz=0.046 0 -0.043 rpy=0 1.8008 0 -> xyz=0.046 0 -0.043 rpy=0 1.770 0
- joint gripper_frame_joint: origin xyz=-0.0079 -0.000218121 -0.0981274 rpy=0 3.14159 0 -> xyz=0.015 0 -0.15 rpy=0 3.14159 0
